File: Board/microcontroller.kicad_sch (KiCad schematic)
At the start: 21 parts, among them J9 ICSP, U2 PIC18F2480-ISO, Y1 10 MHz

Commit message: Rename VPP signal
Connections:
- net VPP_~{MCLR} renamed VPP
Changed lines of the file:
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@@
 		)
 	)
-	(label "VPP_~{MCLR}"
-		(at 121.92 124.46 0)
+	(label "VPP"
+		(at 127 124.46 0)
 		(fields_autoplaced yes)
 		(effects

Commit message: Remove diode in MCU supply line so MCU has full 5V.
Parts:
- removed D5: SS14, Diode_SMD:D_SMA, symbol Device:D_Schottky
Connections:
- net VCC_PIC is gone; now on net VCC: C11.1, J9.2 (Pin_2), U2.20 (VDD)
Changed lines of the file:
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@@
-	)
-	(symbol
-		(lib_id "Device:D_Schottky")
-		(at 80.01 36.83 90)
-		(unit 1)
-		(exclude_from_sim no)
-		(in_bom yes)
-		(on_board yes)
-		(dnp no)
-		(property "Reference" "D5"
-			(at 77.47 34.29 0)
-			(effects
-				(font
-					(size 1.27 1.27)
-				)
-			)
-		)
-		(property "Value" "SS14"
-			(at 77.47 39.37 0)
-			(effects
-				(font
-					(size 1.27 1.27)
-				)
-			)
-		)
-		(property "Footprint" "Diode_SMD:D_SMA"
-			(at 80.01 36.83 0)
-			(effects
-				(font
-					(size 1.27 1.27)
-				)
-				(hide yes)
-			)
-		)
-		(property "Datasheet" "~"
-			(at 80.01 36.83 0)
-			(effects
-				(font
-					(size 1.27 1.27)
-				)
-				(hide yes)
-			)
-		)
-		(property "Description" ""
-			(at 80.01 36.83 0)
-			(effects
-				(font
-					(size 1.27 1.27)
-				)
-				(hide yes)
-			)
-		)
-		(pin "1"
-		)
-		(pin "2"
-		)
-		(instances
-			(project "12VSupport"
-				(path "/f0c44745-560b-4dea-806a-2541c74a511b/3945f109-57ed-41f6-8253-6d6ba9eb298d"
-					(reference "D5")
-					(unit 1)
-				)
-			)
-		)
 	)
 	(symbol
@@
 	(symbol
 		(lib_id "power:VCC")
-		(at 80.01 33.02 0)
+		(at 80.01 40.64 0)
 		(unit 1)
 		(exclude_from_sim no)
@@
 		(fields_autoplaced yes)
 		(property "Reference" "#PWR030"
-			(at 80.01 36.83 0)
+			(at 80.01 44.45 0)
 			(effects
 				(font
@@
 		)
 		(property "Value" "VCC"
-			(at 80.01 27.94 0)
+			(at 80.01 35.56 0)
 			(effects
 				(font
@@
 		)
 		(property "Footprint" ""
-			(at 80.01 33.02 0)
+			(at 80.01 40.64 0)
 			(effects
 				(font
@@
 		)
 		(property "Datasheet" ""
-			(at 80.01 33.02 0)
+			(at 80.01 40.64 0)
 			(effects
 				(font
@@
 		)
 		(property "Description" "Power symbol creates a global label with name \"VCC\""
-			(at 80.01 33.02 0)
+			(at 80.01 40.64 0)
 			(effects
 				(font

Commit message: Board WIP
Parts:
- added C12: 100u, Capacitor_THT:CP_Radial_D6.3mm_P2.50mm, symbol Device:C_Polarized
- added L3: 3u, spetry:CD43, symbol Device:L
Connections:
- net GND: now also C12.2
- net VCC: now also L3.1; no longer C11.1, J9.2 (Pin_2), U2.20 (VDD)
- new net VCC_PIC: C11.1, C12.1, J9.2 (Pin_2), L3.2, U2.20 (VDD)

Commit message: Rev 1.0
Parts:
- added R23: 22K, Resistor_SMD:R_0805_2012Metric, symbol Device:R
Connections:
- net VCC_PIC: now also R23.1
- net VPP: now also R23.2
Other:
- moved on the sheet: C11, C12, C15, C17, D10, D11, D12, D13, D6, D7, D9, J9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

Commit message: WIP
Connections:
- net REL_BOOST_IN: now also U2.15 (SDI/SDA/RC4); no longer U2.12 (T1OSI/RC1)
- new net EN_BOOST_IN: U2.12 (T1OSI/RC1)
- no-connect marks 5 -> 4
Changed lines of the file:
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@@
-	)
-	(no_connect
-		(at 107.95 80.01)
 	)
 	(no_connect
@@
 		(pts
 			(xy 175.26 134.62) (xy 175.26 110.49)
+		)
+		(stroke
+			(width 0)
+			(type default)
+		)
+	)
+	(wire
+		(pts
+			(xy 105.41 80.01) (xy 107.95 80.01)
 		)
 		(stroke
@@
 		)
 	)
-	(global_label "REL_BOOST_IN"
+	(global_label "EN_BOOST_IN"
 		(shape output)
 		(at 105.41 72.39 180)
@@
 		)
 		(property "Intersheetrefs" "${INTERSHEET_REFS}"
-			(at 88.9991 72.39 0)
+			(at 89.9667 72.39 0)
 			(effects
 				(font
@@
 				(hide yes)
 			)
+		)
+	)
+	(global_label "REL_BOOST_IN"
+		(shape output)
+		(at 105.41 80.01 180)
+		(fields_autoplaced yes)
+		(effects
+			(font
+				(size 1.27 1.27)
+			)
+			(justify right)
+		)
+		(property "Intersheetrefs" "${INTERSHEET_REFS}"
+			(at 88.9991 80.01 0)
+			(effects
+				(font
+					(size 1.27 1.27)
+				)
+				(justify right)
+				(hide yes)
+			)
