File: Board/12VSupport.kicad_sch (KiCad schematic)
At the start: 36 parts, among them J1 12V, J2 BATT, J3 BUCK_IN, J4 BUCK_OUT, J5 BOOST_IN, J6 BOOST_OUT, J8 HEATER, K1 SLA-05VDC-SL-C, K2 SLA-05VDC-SL-C, K3 SLA-05VDC-SL-C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

Commit message: Schematic/layout improvements.
Parts:
- added D14, D5: SS14, Diode_SMD:D_SMA, symbol Device:D_Schottky
- added D15: POWER, LED_SMD:LED_0805_2012Metric, symbol Device:LED
- added R19: 680, Resistor_SMD:R_0805_2012Metric, symbol Device:R
Connections:
- net +12V: now also D5.2 (A); no longer C2.1, C5.1, U1.1 (VIN)
- net BUCK_OUT+: now also D14.2 (A)
- net GND: now also D15.1 (K)
- net VCC: now also R19.1
- new net: D15.2 (A), R19.2
- new net: C2.1, C5.1, D14.1 (K), D5.1 (K), U1.1 (VIN)
Other:
- moved on the sheet: Q6

Commit message: Minor improvements
Parts:
- R24: value 10K -> 4K7
Changed lines of the file:
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@@
 			)
 		)
-		(property "Value" "10K"
+		(property "Value" "4K7"
 			(at 195.453 55.372 0)
 			(effects

Commit message: Larger screw terminals.
Parts:
- J1, J2, J3, J4, J5, J6: footprint TerminalBlock:TerminalBlock_Altech_AK300-2_P5.00mm -> spetry:KF7.62_2P
Changed lines of the file:
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@@
 			)
 		)
-		(property "Footprint" "TerminalBlock:TerminalBlock_Altech_AK300-2_P5.00mm"
+		(property "Footprint" "spetry:KF7.62_2P"
 			(at 19.05 147.32 0)
 			(effects
@@
 			)
 		)
-		(property "Footprint" "TerminalBlock:TerminalBlock_Altech_AK300-2_P5.00mm"
+		(property "Footprint" "spetry:KF7.62_2P"
 			(at 120.65 114.3 0)
 			(effects
@@
 			)
 		)
-		(property "Footprint" "TerminalBlock:TerminalBlock_Altech_AK300-2_P5.00mm"
+		(property "Footprint" "spetry:KF7.62_2P"
 			(at 144.78 91.44 0)
 			(effects
@@
 			)
 		)
-		(property "Footprint" "TerminalBlock:TerminalBlock_Altech_AK300-2_P5.00mm"
+		(property "Footprint" "spetry:KF7.62_2P"
 			(at 19.05 116.84 0)
 			(effects
@@
 			)
 		)
-		(property "Footprint" "TerminalBlock:TerminalBlock_Altech_AK300-2_P5.00mm"
+		(property "Footprint" "spetry:KF7.62_2P"
 			(at 120.65 146.05 0)
 			(effects
@@
 			)
 		)
-		(property "Footprint" "TerminalBlock:TerminalBlock_Altech_AK300-2_P5.00mm"
+		(property "Footprint" "spetry:KF7.62_2P"
 			(at 144.78 105.41 0)
 			(effects
