File: Board/sensors.kicad_sch (KiCad schematic)
At the start: 17 parts, among them J7 TMP36GZ, U5 LM324

Commit message: Minor improvements
Connections:
- net BUCK+ renamed B+
- net BUCK- renamed B-
Changed lines of the file:
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@@
 		)
 	)
-	(global_label "BUCK-"
+	(global_label "B-"
 		(shape input)
 		(at 130.81 40.64 180)
@@
 		)
 		(property "Intersheetrefs" "${INTERSHEET_REFS}"
-			(at 121.1119 40.64 0)
+			(at 124.9824 40.64 0)
 			(effects
 				(font
@@
 		)
 	)
-	(global_label "BUCK+"
+	(global_label "B+"
 		(shape input)
 		(at 130.81 45.72 180)
@@
 		)
 		(property "Intersheetrefs" "${INTERSHEET_REFS}"
-			(at 121.1119 45.72 0)
+			(at 124.9824 45.72 0)
 			(effects
 				(font

Commit message: Bugfixes
Parts:
- added R20: 33K, Resistor_SMD:R_0805_2012Metric, symbol Device:R
Connections:
- net 12V_SENSE: now also U5.9 (-); no longer U5.10 (+)
- net GND: now also R20.2
- net at C7.1, J7.2 (Pin_2), U5.12 (+): now also R20.1
- net at C6.1, R5.2, R6.1: now also U5.10 (+); no longer U5.9 (-)
Other:
- moved on the sheet: J7
Changed lines of the file:
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@@
+	)
+	(junction
+		(at 38.1 82.55)
+		(diameter 0)
+		(color 0 0 0 0)
 	)
 	(junction
@@
 	(wire
 		(pts
-			(xy 40.64 82.55) (xy 49.53 82.55)
+			(xy 24.13 82.55) (xy 38.1 82.55)
 		)
 		(stroke
@@
 	(wire
 		(pts
+			(xy 38.1 99.06) (xy 38.1 105.41)
+		)
+		(stroke
+			(width 0)
+			(type default)
+		)
+	)
+	(wire
+		(pts
 			(xy 67.31 52.07) (xy 67.31 45.72)
 		)
@@
 	(wire
 		(pts
+			(xy 38.1 82.55) (xy 38.1 91.44)
+		)
+		(stroke
+			(width 0)
+			(type default)
+		)
+	)
+	(wire
+		(pts
 			(xy 171.45 43.18) (xy 173.99 43.18)
 		)
@@
 	(wire
 		(pts
-			(xy 40.64 80.01) (xy 43.18 80.01)
+			(xy 24.13 80.01) (xy 26.67 80.01)
 		)
 		(stroke
@@
 	(wire
 		(pts
-			(xy 40.64 85.09) (xy 43.18 85.09)
+			(xy 24.13 85.09) (xy 26.67 85.09)
 		)
 		(stroke
@@
 	(wire
 		(pts
+			(xy 38.1 82.55) (xy 49.53 82.55)
+		)
+		(stroke
+			(width 0)
+			(type default)
+		)
+	)
+	(wire
+		(pts
 			(xy 199.39 40.64) (xy 200.66 40.64)
 		)
@@
 	(wire
 		(pts
-			(xy 43.18 85.09) (xy 43.18 87.63)
+			(xy 26.67 85.09) (xy 26.67 87.63)
 		)
 		(stroke
@@
 	(wire
 		(pts
-			(xy 43.18 77.47) (xy 43.18 80.01)
+			(xy 26.67 77.47) (xy 26.67 80.01)
 		)
 		(stroke
@@
 	(symbol
 		(lib_id "power:VCC")
-		(at 43.18 77.47 0)
+		(at 26.67 77.47 0)
 		(unit 1)
 		(exclude_from_sim no)
@@
 		(fields_autoplaced yes)
 		(property "Reference" "#PWR014"
-			(at 43.18 81.28 0)
+			(at 26.67 81.28 0)
 			(effects
 				(font
@@
 		)
 		(property "Value" "VCC"
-			(at 43.18 72.39 0)
+			(at 26.67 72.39 0)
 			(effects
 				(font
@@
 		)
 		(property "Footprint" ""
-			(at 43.18 77.47 0)
+			(at 26.67 77.47 0)
 			(effects
 				(font
@@
 		)
 		(property "Datasheet" ""
-			(at 43.18 77.47 0)
+			(at 26.67 77.47 0)
 			(effects
 				(font
@@
 		)
 		(property "Description" "Power symbol creates a global label with name \"VCC\""
-			(at 43.18 77.47 0)
+			(at 26.67 77.47 0)
 			(effects
 				(font
@@
 	)
 	(symbol
+		(lib_id "Device:R")
+		(at 38.1 95.25 0)
+		(unit 1)
+		(exclude_from_sim no)
+		(in_bom yes)
+		(on_board yes)
+		(dnp no)
+		(fields_autoplaced yes)
+		(property "Reference" "R20"
+			(at 40.64 93.9799 0)
+			(effects
+				(font
+					(size 1.27 1.27)
+				)
+				(justify left)
+			)
+		)
+		(property "Value" "33K"
+			(at 40.64 96.5199 0)
+			(effects
+				(font
+					(size 1.27 1.27)
+				)
+				(justify left)
+			)
+		)
+		(property "Footprint" "Resistor_SMD:R_0805_2012Metric"
+			(at 36.322 95.25 90)
+			(effects
+				(font
+					(size 1.27 1.27)
+				)
+				(hide yes)
+			)
+		)
+		(property "Datasheet" "~"
+			(at 38.1 95.25 0)
+			(effects
+				(font
+					(size 1.27 1.27)
+				)
+				(hide yes)
+			)
+		)
+		(property "Description" "Resistor"
+			(at 38.1 95.25 0)
+			(effects
+				(font
+					(size 1.27 1.27)
+				)
+				(hide yes)
+			)
+		)
+		(pin "1"
+		)
+		(pin "2"
+		)
+		(instances
+			(project "12VSupport"
+				(path "/f0c44745-560b-4dea-806a-2541c74a511b/0c92f1f4-50e9-4520-bdc5-cd5ec6c5b348"
+					(reference "R20")
+					(unit 1)
+				)
+			)
+		)
+	)
+	(symbol
 		(lib_id "Device:L_Ferrite")
 		(at 49.53 129.54 180)
@@
 	(symbol
 		(lib_id "power:GND")
+		(at 38.1 105.41 0)
+		(unit 1)
+		(exclude_from_sim no)
+		(in_bom yes)
+		(on_board yes)
+		(dnp no)
+		(fields_autoplaced yes)
+		(property "Reference" "#PWR019"
+			(at 38.1 111.76 0)
+			(effects
+				(font
+					(size 1.27 1.27)
+				)
+				(hide yes)
+			)
+		)
+		(property "Value" "GND"
+			(at 38.1 110.49 0)
+			(effects
+				(font
+					(size 1.27 1.27)
+				)
+			)
+		)
+		(property "Footprint" ""
+			(at 38.1 105.41 0)
+			(effects
+				(font
+					(size 1.27 1.27)
+				)
+				(hide yes)
+			)
+		)
+		(property "Datasheet" ""
+			(at 38.1 105.41 0)
+			(effects
+				(font
+					(size 1.27 1.27)
+				)
+				(hide yes)
+			)
+		)
+		(property "Description" "Power symbol creates a global label with name \"GND\" , ground"
+			(at 38.1 105.41 0)
+			(effects
+				(font
+					(size 1.27 1.27)
+				)
+				(hide yes)
+			)
+		)
+		(pin "1"
+		)
+		(instances
+			(project "12VSupport"
+				(path "/f0c44745-560b-4dea-806a-2541c74a511b/0c92f1f4-50e9-4520-bdc5-cd5ec6c5b348"
+					(reference "#PWR019")
+					(unit 1)
+				)
+			)
+		)
+	)
+	(symbol
+		(lib_id "power:GND")
 		(at 74.93 113.03 0)
 		(unit 1)
@@
 	(symbol
 		(lib_id "power:GND")
-		(at 43.18 87.63 0)
+		(at 26.67 87.63 0)
 		(unit 1)
 		(exclude_from_sim no)
@@
 		(fields_autoplaced yes)
 		(property "Reference" "#PWR013"
-			(at 43.18 93.98 0)
+			(at 26.67 93.98 0)
 			(effects
 				(font
@@
 		)
 		(property "Value" "GND"
-			(at 43.18 92.71 0)
+			(at 26.67 92.71 0)
 			(effects
 				(font
@@
 		)
 		(property "Footprint" ""
-			(at 43.18 87.63 0)
+			(at 26.67 87.63 0)
 			(effects
 				(font
@@
 		)
 		(property "Datasheet" ""
-			(at 43.18 87.63 0)
+			(at 26.67 87.63 0)
 			(effects
 				(font
@@
 		)
 		(property "Description" "Power symbol creates a global label with name \"GND\" , ground"
-			(at 43.18 87.63 0)
+			(at 26.67 87.63 0)
 			(effects
 				(font
@@
 		(lib_id "Amplifier_Operational:LM324")
 		(at 77.47 43.18 0)
-		(mirror x)
 		(unit 3)
 		(exclude_from_sim no)
@@
 		(dnp no)
 		(property "Reference" "U5"
-			(at 77.47 38.1 0)
+			(at 77.47 48.26 0)
 			(effects
 				(font
@@
 		)
 		(property "Value" "LM324"
-			(at 77.47 48.768 0)
+			(at 77.47 37.592 0)
 			(effects
 				(font
@@
 		)
 		(property "Footprint" "Package_SO:SOIC-14_3.9x8.7mm_P1.27mm"
-			(at 76.2 45.72 0)
+			(at 76.2 40.64 0)
 			(effects
 				(font
@@
 		)
 		(property "Datasheet" "http://www.ti.com/lit/ds/symlink/lm2902-n.pdf"
-			(at 78.74 48.26 0)
+			(at 78.74 38.1 0)
 			(effects
 				(font
@@
 	(symbol
 		(lib_id "Connector:Conn_01x03_Pin")
-		(at 35.56 82.55 0)
+		(at 19.05 82.55 0)
 		(unit 1)
 		(exclude_from_sim no)
@@
 		(fields_autoplaced yes)
 		(property "Reference" "J7"
-			(at 36.195 74.93 0)
+			(at 19.685 74.93 0)
 			(effects
 				(font
@@
 		)
 		(property "Value" "TMP36GZ"
-			(at 36.195 77.47 0)
+			(at 19.685 77.47 0)
 			(effects
 				(font
@@
 		)
 		(property "Footprint" "Connector_PinHeader_2.54mm:PinHeader_1x03_P2.54mm_Vertical"
-			(at 35.56 82.55 0)
+			(at 19.05 82.55 0)
 			(effects
 				(font
@@
 		)
 		(property "Datasheet" "~"
-			(at 35.56 82.55 0)
+			(at 19.05 82.55 0)
 			(effects
 				(font
@@
 		)
 		(property "Description" "Generic connector, single row, 01x03, script generated"
-			(at 35.56 82.55 0)
-			(effects
-				(font
+			(at 19.05 82.55 0)
+			(effects
+				(font

Commit message: Set version number to 1.2. Various fixes. Add fan connector.
Connections:
- net +12V: no longer L2.2
- new net VDD: L2.2
Changed lines of the file:
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@@
 	(title_block
 		(date "2025-01-05")
-		(rev "1.1")
+		(rev "1.2")
 	)
 	(junction
@@
 	)
 	(symbol
-		(lib_id "power:+12V")
-		(at 49.53 125.73 0)
-		(unit 1)
-		(exclude_from_sim no)
-		(in_bom yes)
-		(on_board yes)
-		(dnp no)
-		(fields_autoplaced yes)
-		(property "Reference" "#PWR021"
-			(at 49.53 129.54 0)
-			(effects
-				(font
-					(size 1.27 1.27)
-				)
-				(hide yes)
-			)
-		)
-		(property "Value" "+12V"
-			(at 49.53 120.65 0)
-			(effects
-				(font
-					(size 1.27 1.27)
-				)
-			)
-		)
-		(property "Footprint" ""
-			(at 49.53 125.73 0)
-			(effects
-				(font
-					(size 1.27 1.27)
-				)
-				(hide yes)
-			)
-		)
-		(property "Datasheet" ""
-			(at 49.53 125.73 0)
-			(effects
-				(font
-					(size 1.27 1.27)
-				)
-				(hide yes)
-			)
-		)
-		(property "Description" "Power symbol creates a global label with name \"+12V\""
-			(at 49.53 125.73 0)
-			(effects
-				(font
-					(size 1.27 1.27)
-				)
-				(hide yes)
-			)
-		)
-		(pin "1"
-		)
-		(instances
-			(project "12VSupport"
-				(path "/f0c44745-560b-4dea-806a-2541c74a511b/0c92f1f4-50e9-4520-bdc5-cd5ec6c5b348"
-					(reference "#PWR021")
-					(unit 1)
-				)
-			)
-		)
-	)
-	(symbol
 		(lib_id "Device:R")
 		(at 55.88 45.72 0)
@@
 					(unit 1)
 				)
+			)
+		)
+	)
+	(symbol
+		(lib_id "power:VDD")
+		(at 49.53 125.73 0)
+		(unit 1)
+		(exclude_from_sim no)
+		(in_bom yes)
+		(on_board yes)
+		(dnp no)
+		(fields_autoplaced yes)
+		(property "Reference" "#PWR021"
+			(at 49.53 129.54 0)
+			(effects
+				(font
+					(size 1.27 1.27)
+				)
+				(hide yes)
+			)
+		)
+		(property "Value" "VDD"
+			(at 49.53 120.65 0)
+			(effects
+				(font
+					(size 1.27 1.27)
+				)
+			)
+		)
+		(property "Footprint" ""
+			(at 49.53 125.73 0)
+			(effects
+				(font
+					(size 1.27 1.27)
+				)
+				(hide yes)
+			)
+		)
+		(property "Datasheet" ""
+			(at 49.53 125.73 0)
+			(effects
+				(font
+					(size 1.27 1.27)
+				)
+				(hide yes)
+			)
+		)
+		(property "Description" "Power symbol creates a global label with name \"VDD\""
+			(at 49.53 125.73 0)
+			(effects
+				(font
+					(size 1.27 1.27)
+				)
+				(hide yes)
+			)
+		)
+		(pin "1"
+		)
+		(instances
+			(project ""
+				(path "/f0c44745-560b-4dea-806a-2541c74a511b/0c92f1f4-50e9-4520-bdc5-cd5ec6c5b348"
+					(reference "#PWR021")
+					(unit 1)
+				)

Commit message: Changed battery temp sensor connector.
Parts:
- J7: footprint Connector_PinHeader_2.54mm:PinHeader_1x03_P2.54mm_Vertical -> Connector_JST:JST_PH_B3B-PH-K_1x03_P2.00mm_Vertical
Changed lines of the file:
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@@
 			)
 		)
-		(property "Footprint" "Connector_PinHeader_2.54mm:PinHeader_1x03_P2.54mm_Vertical"
+		(property "Footprint" "Connector_JST:JST_PH_B3B-PH-K_1x03_P2.00mm_Vertical"
 			(at 19.05 82.55 0)
 			(effects

Commit message: Bugfixes
Parts:
- C7: value 47n -> 10n
Connections:
- net +12V renamed SYS_VOLTAGE
- net B+ renamed BAT+
- net B- renamed BAT-
Changed lines of the file:
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@@
 	(wire
 		(pts
-			(xy 55.88 30.48) (xy 55.88 29.21)
+			(xy 55.88 26.67) (xy 55.88 30.48)
 		)
 		(stroke
@@
 		(pts
 			(xy 38.1 137.16) (xy 38.1 135.89)
+		)
+		(stroke
+			(width 0)
+			(type default)
+		)
+	)
+	(wire
+		(pts
+			(xy 55.88 26.67) (xy 59.69 26.67)
 		)
 		(stroke
@@
 		)
 	)
-	(global_label "B-"
+	(global_label "BAT-"
 		(shape input)
 		(at 130.81 40.64 180)
@@
 		)
 		(property "Intersheetrefs" "${INTERSHEET_REFS}"
-			(at 124.9824 40.64 0)
+			(at 122.9262 40.64 0)
 			(effects
 				(font
@@
 		)
 	)
-	(global_label "B+"
+	(global_label "BAT+"
 		(shape input)
 		(at 130.81 45.72 180)
@@
 		)
 		(property "Intersheetrefs" "${INTERSHEET_REFS}"
-			(at 124.9824 45.72 0)
+			(at 122.9262 45.72 0)
 			(effects
 				(font
@@
 				)
 				(justify right)
+				(hide yes)
+			)
+		)
+	)
+	(global_label "SYS_VOLTAGE"
+		(shape input)
+		(at 59.69 26.67 0)
+		(fields_autoplaced yes)
+		(effects
+			(font
+				(size 1.27 1.27)
+			)
+			(justify left)
+		)
+		(property "Intersheetrefs" "${INTERSHEET_REFS}"
+			(at 75.0728 26.67 0)
+			(effects
+				(font
+					(size 1.27 1.27)
+				)
+				(justify left)
 				(hide yes)
 			)
@@
 			)
 		)
-		(property "Value" "47n"
+		(property "Value" "10n"
 			(at 53.34 102.8699 0)
 			(effects
@@
 					(unit 1)
 				)
-			)
-		)
-	)
-	(symbol
-		(lib_id "power:+12V")
-		(at 55.88 29.21 0)
-		(unit 1)
-		(exclude_from_sim no)
-		(in_bom yes)
-		(on_board yes)
-		(dnp no)
-		(fields_autoplaced yes)
-		(property "Reference" "#PWR012"
-			(at 55.88 33.02 0)
-			(effects
-				(font
-					(size 1.27 1.27)
-				)
-				(hide yes)
-			)
-		)
-		(property "Value" "+12V"
-			(at 55.88 24.13 0)
-			(effects
-				(font
-					(size 1.27 1.27)
-				)
-			)
-		)
-		(property "Footprint" ""
-			(at 55.88 29.21 0)
-			(effects
-				(font
-					(size 1.27 1.27)
-				)
-				(hide yes)
-			)
-		)
-		(property "Datasheet" ""
-			(at 55.88 29.21 0)
-			(effects
-				(font
-					(size 1.27 1.27)
-				)
-				(hide yes)
-			)
-		)
-		(property "Description" "Power symbol creates a global label with name \"+12V\""
-			(at 55.88 29.21 0)
-			(effects
-				(font
-					(size 1.27 1.27)
-				)
-				(hide yes)
-			)
-		)
-		(pin "1"
-		)
-		(instances
-			(project "12VSupport"
-				(path "/f0c44745-560b-4dea-806a-2541c74a511b/0c92f1f4-50e9-4520-bdc5-cd5ec6c5b348"
-					(reference "#PWR012")
-					(unit 1)
-				)

Commit message: Bugfixes
Parts:
- added C16: 100n, Capacitor_SMD:C_0805_2012Metric, symbol Device:C
- C9: value 100u -> 220u; footprint Capacitor_SMD:CP_Elec_6.3x7.7 -> Capacitor_THT:CP_Radial_D6.3mm_P2.50mm
Connections:
- net GND: now also C16.2
- net VCC renamed VCC_MCU
- net VCC_MCU: now also C16.1
Other:
- moved on the sheet: C7, C8, C9, L2, R2, R20, R3, R4, U5D, U5E

Commit message: New layout
Parts:
- C9: value 220u -> 100u; footprint Capacitor_THT:CP_Radial_D6.3mm_P2.50mm -> Capacitor_THT:CP_Radial_D5.0mm_P2.50mm
Changed lines of the file:
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@@
 			)
 		)
-		(property "Value" "220u"
+		(property "Value" "100u"
 			(at 58.42 162.9409 0)
 			(effects
@@
 			)
 		)
-		(property "Footprint" "Capacitor_THT:CP_Radial_D6.3mm_P2.50mm"
+		(property "Footprint" "Capacitor_THT:CP_Radial_D5.0mm_P2.50mm"
 			(at 55.5752 166.37 0)
 			(effects
